Commit message: the controlled robot version

File: install/my_car_description/share/my_car_description/urdf/simple_car.urdf.xacro (robot description, xacro)
@@ -7,5 +7,15 @@
   <xacro:property name="base_width" value="0.3"/>
   <xacro:property name="base_height" value="0.1"/>
-  <xacro:property name="wheel_separation_length" value="0.3"/> <!-- Distance between front and rear wheels -->
+  <xacro:property name="wheel_separation_length" value="0.3"/>
+  <!-- Add a dummy base_footprint link to avoid KDL warning -->
+  <link name="base_footprint">
+    <!-- This link has no physical representation, it's just for KDL -->
+  </link>
+  <!-- Connect base_footprint to base_link -->
+  <joint name="base_footprint_joint" type="fixed">
+    <parent link="base_footprint"/>
+    <child link="base_link"/>
+    <origin xyz="0 0 ${wheel_radius}" rpy="0 0 0"/>
+  </joint>
   <!-- Base Link -->
   <link name="base_link">
@@ -28,190 +38,72 @@
     </inertial>
   </link>
-  <!-- Rear Wheels -->
-  <link name="rear_left_wheel">
-    <visual>
-      <geometry>
-        <cylinder radius="${wheel_radius}" length="${wheel_width}"/>
-      </geometry>
-      <origin xyz="0 0 0" rpy="1.5708 0 0"/>
-    </visual>
-    <collision>
-      <geometry>
-        <cylinder radius="${wheel_radius}" length="${wheel_width}"/>
-      </geometry>
-    </collision>
-    <inertial>
-      <mass value="0.5"/>
-      <inertia ixx="0.001" iyy="0.001" izz="0.001" ixy="0" ixz="0" iyz="0"/>
-    </inertial>
-  </link>
-  <link name="rear_right_wheel">
-    <visual>
-      <geometry>
-        <cylinder radius="${wheel_radius}" length="${wheel_width}"/>
-      </geometry>
-      <origin xyz="0 0 0" rpy="1.5708 0 0"/>
-    </visual>
-    <collision>
-      <geometry>
-        <cylinder radius="${wheel_radius}" length="${wheel_width}"/>
-      </geometry>
-    </collision>
-    <inertial>
-      <mass value="0.5"/>
-      <inertia ixx="0.001" iyy="0.001" izz="0.001" ixy="0" ixz="0" iyz="0"/>
-    </inertial>
-  </link>
-  <!-- Front Wheels -->
-  <link name="front_left_wheel">
-    <visual>
-      <geometry>
-        <cylinder radius="${wheel_radius}" length="${wheel_width}"/>
-      </geometry>
-      <origin xyz="0 0 0" rpy="1.5708 0 0"/>
-    </visual>
-    <collision>
-      <geometry>
-        <cylinder radius="${wheel_radius}" length="${wheel_width}"/>
-      </geometry>
-    </collision>
-    <inertial>
-      <mass value="0.5"/>
-      <inertia ixx="0.001" iyy="0.001" izz="0.001" ixy="0" ixz="0" iyz="0"/>
-    </inertial>
-  </link>
-  <link name="front_right_wheel">
-    <visual>
-      <geometry>
-        <cylinder radius="${wheel_radius}" length="${wheel_width}"/>
-      </geometry>
-      <origin xyz="0 0 0" rpy="1.5708 0 0"/>
-    </visual>
-    <collision>
-      <geometry>
-        <cylinder radius="${wheel_radius}" length="${wheel_width}"/>
-      </geometry>
-    </collision>
-    <inertial>
-      <mass value="0.5"/>
-      <inertia ixx="0.001" iyy="0.001" izz="0.001" ixy="0" ixz="0" iyz="0"/>
-    </inertial>
-  </link>
+  <!-- Wheel Definitions -->
+  <xacro:macro name="wheel" params="wheel_name">
+    <link name="${wheel_name}">
+      <visual>
+        <geometry>
+          <cylinder radius="${wheel_radius}" length="${wheel_width}"/>
+        </geometry>
+        <origin xyz="0 0 0" rpy="1.5708 0 0"/>
+      </visual>
+      <collision>
+        <geometry>
+          <cylinder radius="${wheel_radius}" length="${wheel_width}"/>
+        </geometry>
+        <origin xyz="0 0 0" rpy="1.5708 0 0"/>
+      </collision>
+      <inertial>
+        <mass value="0.5"/>
+        <inertia ixx="0.001" iyy="0.001" izz="0.001" ixy="0" ixz="0" iyz="0"/>
+      </inertial>
+    </link>
+  </xacro:macro>
+  <xacro:wheel wheel_name="rear_left_wheel"/>
+  <xacro:wheel wheel_name="rear_right_wheel"/>
+  <xacro:wheel wheel_name="front_left_wheel"/>
+  <xacro:wheel wheel_name="front_right_wheel"/>
   <!-- Joints -->
-  <!-- Rear Wheels Joints -->
-  <joint name="rear_left_wheel_joint" type="continuous">
-    <parent link="base_link"/>
-    <child link="rear_left_wheel"/>
-    <origin xyz="-${wheel_separation_length/2} ${base_width/2} -${wheel_radius}" rpy="0 0 0"/>
-    <axis xyz="0 1 0"/>
-  </joint>
-  <joint name="rear_right_wheel_joint" type="continuous">
-    <parent link="base_link"/>
-    <child link="rear_right_wheel"/>
-    <origin xyz="-${wheel_separation_length/2} -${base_width/2} -${wheel_radius}" rpy="0 0 0"/>
-    <axis xyz="0 1 0"/>
-  </joint>
-  <!-- Front Wheels Joints -->
-  <joint name="front_left_wheel_joint" type="continuous">
-    <parent link="base_link"/>
-    <child link="front_left_wheel"/>
-    <origin xyz="${wheel_separation_length/2} ${base_width/2} -${wheel_radius}" rpy="0 0 0"/>
-    <axis xyz="0 1 0"/>
-  </joint>
-  <joint name="front_right_wheel_joint" type="continuous">
-    <parent link="base_link"/>
-    <child link="front_right_wheel"/>
-    <origin xyz="${wheel_separation_length/2} -${base_width/2} -${wheel_radius}" rpy="0 0 0"/>
-    <axis xyz="0 1 0"/>
-  </joint>
-  <!-- Sonar Sensor -->
+  <xacro:macro name="wheel_joint" params="parent_link child_link joint_name x y z">
+    <joint name="${joint_name}" type="continuous">
+      <parent link="${parent_link}"/>
+      <child link="${child_link}"/>
+      <origin xyz="${x} ${y} ${z}" rpy="0 0 0"/>
+      <axis xyz="0 1 0"/>
+    </joint>
+  </xacro:macro>
+  <xacro:wheel_joint parent_link="base_link" child_link="rear_left_wheel" joint_name="rear_left_wheel_joint" x="-0.15" y="0.15" z="-0.05"/>
+  <xacro:wheel_joint parent_link="base_link" child_link="rear_right_wheel" joint_name="rear_right_wheel_joint" x="-0.15" y="-0.15" z="-0.05"/>
+  <xacro:wheel_joint parent_link="base_link" child_link="front_left_wheel" joint_name="front_left_wheel_joint" x="0.15" y="0.15" z="-0.05"/>
+  <xacro:wheel_joint parent_link="base_link" child_link="front_right_wheel" joint_name="front_right_wheel_joint" x="0.15" y="-0.15" z="-0.05"/>
+  <!-- Gazebo material colors -->
   <gazebo reference="base_link">
-    <sensor type="ray" name="sonar_sensor">
-      <pose>0 0 0.15 0 0 0</pose>
-      <ray>
-        <scan>
-          <horizontal>
-            <samples>1</samples>
-            <resolution>1.0</resolution>
-            <min_angle>0</min_angle>
-            <max_angle>0</max_angle>
-          </horizontal>
-        </scan>
-        <range>
-          <min>0.05</min>
-          <max>2.0</max>
-          <resolution>0.01</resolution>
-        </range>
-      </ray>
-      <plugin name="gazebo_ros_range" filename="libgazebo_ros_range.so">
-        <ros>
-          <remapping>~/out:=/distance</remapping>
-        </ros>
-        <frameName>base_link</frameName>
-      </plugin>
-    </sensor>
+    <material>Gazebo/Blue</material>
   </gazebo>
-  <!-- ROS2 Control -->
-  <ros2_control name="MyCarControl" type="system">
-    <hardware>
-      <plugin>gazebo_ros2_control/GazeboSystem</plugin>
-    </hardware>
-    <joint name="rear_left_wheel_joint">
-      <command_interface name="velocity"/>
-      <state_interface name="velocity"/>
-    </joint>
-    <joint name="rear_right_wheel_joint">
-      <command_interface name="velocity"/>
-      <state_interface name="velocity"/>
-    </joint>
-    <joint name="front_left_wheel_joint">
-      <command_interface name="velocity"/>
-      <state_interface name="velocity"/>
-    </joint>
-    <joint name="front_right_wheel_joint">
-      <command_interface name="velocity"/>
-      <state_interface name="velocity"/>
-    </joint>
-  </ros2_control>
-  <!-- Transmissions -->
-  <transmission name="rear_left_wheel_trans">
-    <type>transmission_interface/SimpleTransmission</type>
-    <joint name="rear_left_wheel_joint">
-      <hardwareInterface>velocity</hardwareInterface>
-    </joint>
-    <actuator name="rear_left_motor">
-      <hardwareInterface>velocity</hardwareInterface>
-      <mechanicalReduction>1</mechanicalReduction>
-    </actuator>
-  </transmission>
-  <transmission name="rear_right_wheel_trans">
-    <type>transmission_interface/SimpleTransmission</type>
-    <joint name="rear_right_wheel_joint">
-      <hardwareInterface>velocity</hardwareInterface>
-    </joint>
-    <actuator name="rear_right_motor">
-      <hardwareInterface>velocity</hardwareInterface>
-      <mechanicalReduction>1</mechanicalReduction>
-    </actuator>
-  </transmission>
-  <transmission name="front_left_wheel_trans">
-    <type>transmission_interface/SimpleTransmission</type>
-    <joint name="front_left_wheel_joint">
-      <hardwareInterface>velocity</hardwareInterface>
-    </joint>
-    <actuator name="front_left_motor">
-      <hardwareInterface>velocity</hardwareInterface>
-      <mechanicalReduction>1</mechanicalReduction>
-    </actuator>
-  </transmission>
-  <transmission name="front_right_wheel_trans">
-    <type>transmission_interface/SimpleTransmission</type>
-    <joint name="front_right_wheel_joint">
-      <hardwareInterface>velocity</hardwareInterface>
-    </joint>
-    <actuator name="front_right_motor">
-      <hardwareInterface>velocity</hardwareInterface>
-      <mechanicalReduction>1</mechanicalReduction>
-    </actuator>
-  </transmission>
+  <gazebo reference="rear_left_wheel">
+    <material>Gazebo/Black</material>
+  </gazebo>
+  <gazebo reference="rear_right_wheel">
+    <material>Gazebo/Black</material>
+  </gazebo>
+  <gazebo reference="front_left_wheel">
+    <material>Gazebo/Black</material>
+  </gazebo>
+  <gazebo reference="front_right_wheel">
+    <material>Gazebo/Black</material>
+  </gazebo>
+  <!-- Diff Drive Plugin - UPDATED for ROS2 -->
+  <gazebo>
+    <plugin name="diff_drive_controller" filename="libgazebo_ros_diff_drive.so">
+      <ros>
+        <remapping>cmd_vel:=/cmd_vel</remapping>
+      </ros>
+      <left_joint>rear_left_wheel_joint</left_joint>
+      <right_joint>rear_right_wheel_joint</right_joint>
+      <wheel_separation>0.3</wheel_separation>
+      <wheel_diameter>0.1</wheel_diameter>
+      <max_wheel_torque>10</max_wheel_torque>
+      <odometry_frame>odom</odometry_frame>
+      <robot_base_frame>base_link</robot_base_frame>
+    </plugin>
+  </gazebo>
 </robot>

Commit message: final version of simulation

File: install/my_car_description/share/my_car_description/urdf/simple_car.urdf.xacro (robot description, xacro)
@@ -76,4 +76,73 @@
   <xacro:wheel_joint parent_link="base_link" child_link="front_left_wheel" joint_name="front_left_wheel_joint" x="0.15" y="0.15" z="-0.05"/>
   <xacro:wheel_joint parent_link="base_link" child_link="front_right_wheel" joint_name="front_right_wheel_joint" x="0.15" y="-0.15" z="-0.05"/>
+  <!-- ✅ SONAR SENSOR -->
+  <link name="sonar_link">
+    <visual>
+      <geometry>
+        <cylinder length="0.05" radius="0.015"/>
+      </geometry>
+      <origin xyz="0 0 0" rpy="0 0 0"/>
+      <material name="gray">
+        <color rgba="0.5 0.5 0.5 1"/>
+      </material>
+    </visual>
+    <collision>
+      <geometry>
+        <cylinder length="0.05" radius="0.015"/>
+      </geometry>
+      <origin xyz="0 0 0" rpy="0 0 0"/>
+    </collision>
+    <inertial>
+      <mass value="0.01"/>
+      <inertia ixx="1e-6" iyy="1e-6" izz="1e-6" ixy="0.0" ixz="0.0" iyz="0.0"/>
+    </inertial>
+  </link>
+  <joint name="sonar_joint" type="fixed">
+    <parent link="base_link"/>
+    <child link="sonar_link"/>
+    <origin xyz="0.17 0 0.065" rpy="0 0 0"/>
+  </joint>
+  <gazebo reference="sonar_link">
+    <sensor type="ray" name="sonar_sensor">
+      <pose>0 0 0 0 0 0</pose>
+      <visualize>true</visualize>
+      <update_rate>10.0</update_rate>
+      <always_on>true</always_on>
+      <ray>
+        <scan>
+          <horizontal>
+            <samples>9</samples>              <!-- More rays for visibility -->
+            <resolution>1.0</resolution>
+            <min_angle>-0.15</min_angle>      <!-- ~17 degree cone -->
+            <max_angle>0.15</max_angle>       <!-- ~17 degree cone -->
+          </horizontal>
+          <vertical>
+            <samples>3</samples>              <!-- Add vertical rays -->
+            <resolution>1.0</resolution>
+            <min_angle>-0.05</min_angle>
+            <max_angle>0.05</max_angle>
+          </vertical>
+        </scan>
+        <range>
+          <min>0.02</min>
+          <max>3.0</max>
+          <resolution>0.01</resolution>
+        </range>
+        <noise>
+          <type>gaussian</type>
+          <mean>0.0</mean>
+          <stddev>0.01</stddev>
+        </noise>
+      </ray>
+      <plugin name="sonar_controller" filename="libgazebo_ros_ray_sensor.so">
+        <ros>
+          <namespace>/</namespace>
+          <remapping>~/out:=/sonar</remapping>
+        </ros>
+        <output_type>sensor_msgs/Range</output_type>
+        <frame_name>sonar_link</frame_name>
+      </plugin>
+    </sensor>
+  </gazebo>
   <!-- Gazebo material colors -->
   <gazebo reference="base_link">
